Commit message: added the segmentation model

File: grp_system_description/urdf/free_camera.xacro (robot description, xacro)
@@ -24,5 +24,5 @@
   <!-- ================= GAZEBO CAMERA SENSOR ================= -->
   <gazebo reference="free_camera_link">
-    <material>Gazebo/Yellow</material>
+    <material>Gazebo/Red</material>
     <!-- <gravity>0</gravity> -->
     <static>false</static>

File: grp_system_description/urdf/ssmr_gazebo_ros2_conrtol.xacro (robot description, xacro)
@@ -3,6 +3,6 @@
     <xacro:macro name="create_joint_tag_ros2_cont" params="prefix">
         <joint name="${prefix}">
-            <!-- <command_interface name="effort"> -->
-            <command_interface name="velocity">
+            <command_interface name="effort">
+            <!-- <command_interface name="velocity"> -->
                 <param name="max">100</param>
                 <param name="min">-100</param>
