Commit message: model uploaded

File: grp_system_description/urdf/ssmr_base.xacro (robot description, xacro)
@@ -75,5 +75,6 @@
         <material>Gazebo/Blue</material>
     </gazebo>
-    <link name="robot_picture">
+    <!-- Aruco marker -->
+    <!-- <link name="robot_picture">
         <visual>
             <geometry>
@@ -89,5 +90,5 @@
         <child link="robot_picture"/>
         <origin xyz="0 0 ${chassis_height/2}" rpy="0 0 0"/>
-    </joint>
+    </joint> -->
     <xacro:wheel prefix="front_left"  x_reflect="1"  y_reflect="1"/>
     <xacro:wheel prefix="front_right" x_reflect="1"  y_reflect="-1"/>

Commit message: new stuff

File: grp_system_description/urdf/ssmr_base.xacro (robot description, xacro)
@@ -39,5 +39,5 @@
         </joint>
         <gazebo reference="${prefix}_wheel">
-            <material>Gazebo/Orange</material>
+            <material>Gazebo/Blue</material>
             <mu1 value="0.2"/>
             <mu2 value="0.2"/>
@@ -76,5 +76,5 @@
     </gazebo>
     <!-- Aruco marker -->
-    <!-- <link name="robot_picture">
+    <link name="robot_picture">
         <visual>
             <geometry>
@@ -90,5 +90,5 @@
         <child link="robot_picture"/>
         <origin xyz="0 0 ${chassis_height/2}" rpy="0 0 0"/>
-    </joint> -->
+    </joint>
     <xacro:wheel prefix="front_left"  x_reflect="1"  y_reflect="1"/>
     <xacro:wheel prefix="front_right" x_reflect="1"  y_reflect="-1"/>

Commit message: added pure pursuit and faild vfg

File: grp_system_description/urdf/ssmr_base.xacro (robot description, xacro)
@@ -76,5 +76,5 @@
     </gazebo>
     <!-- Aruco marker -->
-    <link name="robot_picture">
+    <!-- <link name="robot_picture">
         <visual>
             <geometry>
@@ -90,5 +90,5 @@
         <child link="robot_picture"/>
         <origin xyz="0 0 ${chassis_height/2}" rpy="0 0 0"/>
-    </joint>
+    </joint> -->
     <xacro:wheel prefix="front_left"  x_reflect="1"  y_reflect="1"/>
     <xacro:wheel prefix="front_right" x_reflect="1"  y_reflect="-1"/>
